File: Solaranlage.sch (KiCad schematic (older format))
At the start: 77 parts, among them J1 Screw_Terminal_01x02, J10 Conn_01x01_Male, J2 Screw_Terminal_01x02, J3 AVR-JTAG-10, J4 USB_B, J5 USB_B, J6 Screw_Terminal_01x02, J7 Conn_01x02_Male, J8 Conn_01x01_Male, J9 Conn_01x02_Male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

Commit message: attached AREF-pin to 5V
Parts:
- gave numbers to parts that had none: 1
Connections:
- wire segments 371 -> 370
Other:
- moved on the sheet: C10, C11, C12, C13, C14, C2, C5, D2, D3, J6, L1, R10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

Commit message: flipped designator C3 and R1 in silk screen
Parts:
- added L2: INDUCTOR, Inductor_THT:L_Radial_D10.0mm_P5.00mm_Fastron_07P, symbol pspice:INDUCTOR
Connections:
- wire segments 370 -> 371
Changed lines of the file:
@@
 Connection ~ 4750 3550
 Wire Wire Line
-	13250 4050 13250 2050
+	13250 4050 13250 3050
 Connection ~ 13250 4050
 $Comp
-L power:+5V #PWR?
+L power:+5V #PWR0115
 U 1 1 5FCF10EB
 P 13250 2050
-F 0 "#PWR?" H 13250 1900 50  0001 C CNN
+F 0 "#PWR0115" H 13250 1900 50  0001 C CNN
 F 1 "+5V" H 13265 2223 50  0000 C CNN
 F 2 "" H 13250 2050 50  0001 C CNN
@@
 	1    0    0    -1
 $EndComp
+$Comp
+L pspice:INDUCTOR L2
+U 1 1 5FD19EB6
+P 13250 2800
+F 0 "L2" V 13204 2756 50  0000 R CNN
+F 1 "INDUCTOR" V 13295 2756 50  0000 R CNN
+F 2 "Inductor_THT:L_Radial_D10.0mm_P5.00mm_Fastron_07P" H 13250 2800 50  0001 C CNN
+F 3 "~" H 13250 2800 50  0001 C CNN
+	1    13250 2800
+	0    1    1    0
+$EndComp
+Wire Wire Line
+	13250 2550 13250 2050
 $EndSCHEMATC

Commit message: fixed reset of ne555
Connections:
- wire segments 371 -> 370
Changed lines of the file:
@@
 	14500 11400 14500 11500
 Wire Wire Line
-	14500 9700 14950 9700
-Wire Wire Line
 	16500 9700 16500 10950
 Wire Wire Line
@@
 Wire Wire Line
 	15100 10950 14950 10950
-Wire Wire Line
-	14950 10950 14950 9700
-Connection ~ 14950 9700
-Wire Wire Line
-	14950 9700 16500 9700
 $Comp
 L power:GND #PWR035
@@
 Wire Wire Line
 	14950 10950 14950 11100
-Connection ~ 14950 10950
 $Comp
 L Device:R R24
@@
 Wire Wire Line
 	13250 2550 13250 2050
+$Comp
+L power:+5V #PWR?
+U 1 1 5FD425B5
+P 14950 9950
+F 0 "#PWR?" H 14950 9800 50  0001 C CNN
+F 1 "+5V" H 14965 10123 50  0000 C CNN
+F 2 "" H 14950 9950 50  0001 C CNN
+F 3 "" H 14950 9950 50  0001 C CNN
+	1    14950 9950
+	1    0    0    -1
+$EndComp
+Wire Wire Line
+	14500 9700 16500 9700
+Wire Wire Line
+	14950 9950 14950 10950
+Connection ~ 14950 10950
 $EndSCHEMATC

Commit message: changed MCU from atmega32 to atmega644 because of availability;added 12p->GND to TCK to make JTAG working
Parts:
- removed Q1: 2N7000, Package_TO_SOT_THT:TO-92_Inline, symbol Transistor_FET:2N7000
- added Q?: 2N3904, Package_TO_SOT_THT:TO-92_Inline, symbol Transistor_BJT:2N3904
- added Q?: BC328, Package_TO_SOT_THT:TO-92_Inline, symbol Transistor_BJT:BC328
Connections:
- wire segments 370 -> 374
Other:
- moved on the sheet: C15, R22, R23
Changed lines of the file:
@@
 Text Label 13350 3650 0    50   ~ 0
 XTAL1
-Text GLabel 16700 10550 2    50   Input ~ 0
+Text GLabel 16650 10550 2    50   Input ~ 0
 \RST
 $Comp
@@
 L power:GND #PWR037
 U 1 1 5F613410
-P 15600 11500
-F 0 "#PWR037" H 15600 11250 50  0001 C CNN
-F 1 "GND" H 15605 11327 50  0000 C CNN
-F 2 "" H 15600 11500 50  0001 C CNN
-F 3 "" H 15600 11500 50  0001 C CNN
-	1    15600 11500
-	1    0    0    -1
-$EndComp
-Wire Wire Line
-	15600 11150 15600 11500
+P 15600 11550
+F 0 "#PWR037" H 15600 11300 50  0001 C CNN
+F 1 "GND" H 15605 11377 50  0000 C CNN
+F 2 "" H 15600 11550 50  0001 C CNN
+F 3 "" H 15600 11550 50  0001 C CNN
+	1    15600 11550
+	1    0    0    -1
+$EndComp
+Wire Wire Line
+	15600 11150 15600 11550
 Wire Wire Line
 	15600 10350 15600 9950
@@
 L power:GND #PWR034
 U 1 1 5F75EEAF
-P 14500 11500
-F 0 "#PWR034" H 14500 11250 50  0001 C CNN
-F 1 "GND" H 14505 11327 50  0000 C CNN
-F 2 "" H 14500 11500 50  0001 C CNN
-F 3 "" H 14500 11500 50  0001 C CNN
-	1    14500 11500
-	1    0    0    -1
-$EndComp
-Wire Wire Line
-	14500 11400 14500 11500
+P 14500 11550
+F 0 "#PWR034" H 14500 11300 50  0001 C CNN
+F 1 "GND" H 14505 11377 50  0000 C CNN
+F 2 "" H 14500 11550 50  0001 C CNN
+F 3 "" H 14500 11550 50  0001 C CNN
+	1    14500 11550
+	1    0    0    -1
+$EndComp
+Wire Wire Line
+	14500 11400 14500 11550
 Wire Wire Line
 	16500 9700 16500 10950
@@
 L power:GND #PWR035
 U 1 1 5F88C218
-P 14950 11500
-F 0 "#PWR035" H 14950 11250 50  0001 C CNN
-F 1 "GND" H 14955 11327 50  0000 C CNN
-F 2 "" H 14950 11500 50  0001 C CNN
-F 3 "" H 14950 11500 50  0001 C CNN
-	1    14950 11500
+P 14950 11550
+F 0 "#PWR035" H 14950 11300 50  0001 C CNN
+F 1 "GND" H 14955 11377 50  0000 C CNN
+F 2 "" H 14950 11550 50  0001 C CNN
+F 3 "" H 14950 11550 50  0001 C CNN
+	1    14950 11550
 	1    0    0    -1
 $EndComp
@@
 L power:GND #PWR033
 U 1 1 5F926C80
-P 14000 11500
-F 0 "#PWR033" H 14000 11250 50  0001 C CNN
-F 1 "GND" H 14005 11327 50  0000 C CNN
-F 2 "" H 14000 11500 50  0001 C CNN
-F 3 "" H 14000 11500 50  0001 C CNN
-	1    14000 11500
+P 14000 11550
+F 0 "#PWR033" H 14000 11300 50  0001 C CNN
+F 1 "GND" H 14005 11377 50  0000 C CNN
+F 2 "" H 14000 11550 50  0001 C CNN
+F 3 "" H 14000 11550 50  0001 C CNN
+	1    14000 11550
 	1    0    0    -1
 $EndComp
@@
 	14000 9950 14000 10150
 Wire Wire Line
-	14000 11400 14000 11500
+	14000 11400 14000 11550
 Wire Wire Line
 	14000 10450 14000 10550
 Wire Wire Line
-	13400 10900 13400 10550
-Wire Wire Line
-	13400 10550 14000 10550
+	12400 10900 12400 10550
+Wire Wire Line
+	12400 10550 13000 10550
 Connection ~ 14000 10550
 Wire Wire Line
@@
 L power:GND #PWR031
 U 1 1 5FA379A1
-P 13400 11550
-F 0 "#PWR031" H 13400 11300 50  0001 C CNN
-F 1 "GND" H 13405 11377 50  0000 C CNN
-F 2 "" H 13400 11550 50  0001 C CNN
-F 3 "" H 13400 11550 50  0001 C CNN
-	1    13400 11550
-	1    0    0    -1
-$EndComp
-Wire Wire Line
-	13400 11300 13400 11550
+P 12400 11550
+F 0 "#PWR031" H 12400 11300 50  0001 C CNN
+F 1 "GND" H 12405 11377 50  0000 C CNN
+F 2 "" H 12400 11550 50  0001 C CNN
+F 3 "" H 12400 11550 50  0001 C CNN
+	1    12400 11550
+	1    0    0    -1
+$EndComp
+Wire Wire Line
+	12400 11300 12400 11550
 $Comp
 L Device:R R22
 U 1 1 5FA86A27
-P 12550 11300
-F 0 "R22" H 12620 11346 50  0000 L CNN
-F 1 "10k" H 12620 11255 50  0000 L CNN
-F 2 "Resistor_THT:R_Axial_DIN0204_L3.6mm_D1.6mm_P7.62mm_Horizontal" H 12620 11209 50  0001 L CNN
-F 3 "~" H 12550 11300 50  0001 C CNN
-	1    12550 11300
+P 11550 11300
+F 0 "R22" H 11350 11350 50  0000 L CNN
+F 1 "10k" H 11350 11250 50  0000 L CNN
+F 2 "Resistor_THT:R_Axial_DIN0204_L3.6mm_D1.6mm_P7.62mm_Horizontal" H 11620 11209 50  0001 L CNN
+F 3 "~" H 11550 11300 50  0001 C CNN
+	1    11550 11300
 	1    0    0    -1
 $EndComp
@@
 L Device:R R23
 U 1 1 5FAAEAC8
-P 12850 11100
-F 0 "R23" V 13050 11100 50  0000 L CNN
-F 1 "1k" V 12950 11050 50  0000 L CNN
-F 2 "Resistor_THT:R_Axial_DIN0204_L3.6mm_D1.6mm_P7.62mm_Horizontal" H 12920 11009 50  0001 L CNN
-F 3 "~" H 12850 11100 50  0001 C CNN
-	1    12850 11100
+P 11850 11100
+F 0 "R23" V 12050 11050 50  0000 L CNN
+F 1 "1k" V 11950 11100 50  0000 L CNN
+F 2 "Resistor_THT:R_Axial_DIN0204_L3.6mm_D1.6mm_P7.62mm_Horizontal" H 11920 11009 50  0001 L CNN
+F 3 "~" H 11850 11100 50  0001 C CNN
+	1    11850 11100
 	0    -1   -1   0
 $EndComp
@@
 L power:GND #PWR030
 U 1 1 5FB26AA0
-P 12550 11550
-F 0 "#PWR030" H 12550 11300 50  0001 C CNN
-F 1 "GND" H 12555 11377 50  0000 C CNN
-F 2 "" H 12550 11550 50  0001 C CNN
-F 3 "" H 12550 11550 50  0001 C CNN
-	1    12550 11550
-	1    0    0    -1
-$EndComp
-Wire Wire Line
-	13100 11100 13000 11100
-Wire Wire Line
-	12700 11100 12550 11100
-Wire Wire Line
-	12550 11100 12550 11150
-Wire Wire Line
-	12550 11450 12550 11550
-Connection ~ 12550 11100
-Wire Wire Line
-	12550 11100 12300 11100
+P 11550 11550
+F 0 "#PWR030" H 11550 11300 50  0001 C CNN
+F 1 "GND" H 11555 11377 50  0000 C CNN
+F 2 "" H 11550 11550 50  0001 C CNN
+F 3 "" H 11550 11550 50  0001 C CNN
+	1    11550 11550
+	1    0    0    -1
+$EndComp
+Wire Wire Line
+	12100 11100 12000 11100
+Wire Wire Line
+	11700 11100 11550 11100
+Wire Wire Line
+	11550 11100 11550 11150
+Wire Wire Line
+	11550 11450 11550 11550
+Connection ~ 11550 11100
+Wire Wire Line
+	11550 11100 11300 11100
 $Comp
 L Device:CP C16
@@
 L Device:C C15
 U 1 1 5FCBD478
-P 12150 11100
-F 0 "C15" H 12265 11146 50  0000 L CNN
-F 1 "10n" H 12265 11055 50  0000 L CNN
-F 2 "Capacitor_THT:C_Rect_L9.0mm_W2.5mm_P7.50mm_MKT" H 12188 10950 50  0001 C CNN
-F 3 "~" H 12150 11100 50  0001 C CNN
-F 4 "" V 11950 11150 50  0001 C CNN "Ordering Code"
-	1    12150 11100
+P 11150 11100
+F 0 "C15" V 11400 11050 50  0000 L CNN
+F 1 "10n" V 11300 11050 50  0000 L CNN
+F 2 "Capacitor_THT:C_Rect_L9.0mm_W2.5mm_P7.50mm_MKT" H 11188 10950 50  0001 C CNN
+F 3 "~" H 11150 11100 50  0001 C CNN
+F 4 "" V 10950 11150 50  0001 C CNN "Ordering Code"
+	1    11150 11100
 	0    -1   -1   0
 $EndComp
 Wire Wire Line
-	12000 11100 11500 11100
-Wire Wire Line
-	16100 10550 16700 10550
+	11000 11100 10750 11100
+Wire Wire Line
+	16100 10550 16650 10550
 Wire Wire Line
 	11300 5850 11950 5850
 Text GLabel 11300 5850 0    50   Output ~ 0
 WDI
-Text GLabel 11500 11100 0    50   Input ~ 0
+Text GLabel 10750 11100 0    50   Input ~ 0
 WDI
-$Comp
-L Transistor_FET:2N7000 Q1
-U 1 1 5F8AC9A0
-P 13300 11100
-F 0 "Q1" H 13504 11146 50  0000 L CNN
-F 1 "2N7000" H 13504 11055 50  0000 L CNN
-F 2 "Package_TO_SOT_THT:TO-92_Inline" H 13500 11025 50  0001 L CIN
-F 3 "https://www.fairchildsemi.com/datasheets/2N/2N7000.pdf" H 13300 11100 50  0001 L CNN
-	1    13300 11100
-	1    0    0    -1
-$EndComp
 $Comp
 L Device:C C1
@@
 $EndComp
 Wire Wire Line
-	14950 11400 14950 11500
+	14950 11400 14950 11550
 $Comp
 L Device:C C17
@@
 	13250 2550 13250 2050
 $Comp
-L power:+5V #PWR?
+L power:+5V #PWR0116
 U 1 1 5FD425B5
 P 14950 9950
-F 0 "#PWR?" H 14950 9800 50  0001 C CNN
+F 0 "#PWR0116" H 14950 9800 50  0001 C CNN
 F 1 "+5V" H 14965 10123 50  0000 C CNN
 F 2 "" H 14950 9950 50  0001 C CNN
@@
 	14950 9950 14950 10950
 Connection ~ 14950 10950
+$Comp
+L power:GND #PWR?
+U 1 1 5FE8332C
+P 13000 11550
+F 0 "#PWR?" H 13000 11300 50  0001 C CNN
+F 1 "GND" H 13005 11377 50  0000 C CNN
+F 2 "" H 13000 11550 50  0001 C CNN
+F 3 "" H 13000 11550 50  0001 C CNN
+	1    13000 11550
+	1    0    0    -1
+$EndComp
+Wire Wire Line
+	13000 11300 13000 11550
+Wire Wire Line
+	13000 10900 13000 10550
+Connection ~ 13000 10550
+Wire Wire Line
+	13000 10550 14000 10550
+Text GLabel 13350 11100 2    50   Input ~ 0
+\RST
+Wire Wire Line
+	13350 11100 13300 11100
+$Comp
+L Transistor_BJT:2N3904 Q?
+U 1 1 5FF728D8
+P 12300 11100
+F 0 "Q?" H 12250 11300 50  0000 L CNN
+F 1 "2N3904" H 12050 10950 50  0000 L CNN
+F 2 "Package_TO_SOT_THT:TO-92_Inline" H 12500 11025 50  0001 L CIN
+F 3 "https://www.fairchildsemi.com/datasheets/2N/2N3904.pdf" H 12300 11100 50  0001 L CNN
+	1    12300 11100
+	1    0    0    -1
+$EndComp
+$Comp
+L Transistor_BJT:BC328 Q?
+U 1 1 5FF9EB7A
+P 13100 11100
+F 0 "Q?" H 13291 11146 50  0000 L CNN
+F 1 "BC328" H 13291 11055 50  0000 L CNN
+F 2 "Package_TO_SOT_THT:TO-92_Inline" H 13300 11025 50  0001 L CIN
+F 3 "http://www.redrok.com/PNP_BC327_-45V_-800mA_0.625W_Hfe100_TO-92.pdf" H 13100 11100 50  0001 L CNN
+	1    13100 11100
+	-1   0    0    -1
+$EndComp
 $EndSCHEMATC

Commit message: added Q2 to watchdog circuit;
Parts:
- removed C17: 10n, Capacitor_THT:C_Rect_L9.0mm_W2.5mm_P7.50mm_MKT, symbol Device:C
- removed U7: ATmega32-16PU, Package_DIP:DIP-40_W15.24mm, symbol MCU_Microchip_ATmega:ATmega32-16PU
- added C19: 10p, Capacitor_THT:C_Disc_D4.7mm_W2.5mm_P5.00mm, symbol Device:C
- added U7: ATmega644-20PU, Package_DIP:DIP-40_W15.24mm, symbol MCU_Microchip_ATmega:ATmega644-20PU
- C12, C13: value 100n -> 10p
- Q1, Q2: renamed from Q?; footprint Package_TO_SOT_THT:TO-92_Inline -> Package_TO_SOT_THT:TO-92_HandSolder
Connections:
- net +5V: now also U7.10 (VCC)
- net A: now also U7.1 (PB0)
- net AREF: now also U7.32 (AREF)
- net AVCC: now also U7.30 (AVCC)
- net B: now also U7.2 (PB1)
- net C: now also U7.3 (PB2)
- net D: now also U7.4 (PB3)
- net DACH_ADC: now also U7.40 (PA0)
- net DE: now also U7.35 (PA5)
- net DH: now also U7.33 (PA7)
- net DP: now also U7.8 (PB7)
- net DZ: now also U7.34 (PA6)
- net E: now also U7.5 (PB4)
- net ENC_A: now also U7.16 (PD2)
- net ENC_B: now also U7.18 (PD4)
- net F: now also U7.6 (PB5)
- net G: now also U7.7 (PB6)
- net GND: now also C19.2, U7.11 (GND), U7.31 (GND)
- net Heart_LED: now also U7.19 (PD5)
- net KE: now also U7.38 (PA2)
- net KELLER_ADC: now also U7.39 (PA1)
- net KH: now also U7.36 (PA4)
- net KZ: now also U7.37 (PA3)
- net PWM: now also U7.21 (PD7)
- net RxD: now also U7.14 (PD0)
- net SW1: now also U7.17 (PD3)
- net TCK: now also C19.1, U7.24 (PC2)
- net TDI: now also U7.27 (PC5)
- net TDO: now also U7.26 (PC4)
- net TMS: now also U7.25 (PC3)
- net TxD: now also U7.15 (PD1)
- net WDI: now also U7.28 (PC6)
- net XTAL1: now also U7.13 (XTAL1)
- net XTAL2: now also U7.12 (XTAL2)
- net \RST: now also U7.9 (~RESET)
Changed lines of the file:
@@
 	21150 5000 21750 5000
 Wire Wire Line
-	21150 4800 21750 4800
+	21150 4800 22500 4800
 Text Notes 20750 4350 1    50   ~ 0
 sould be left N.C.\n
@@
 Wire Wire Line
 	21150 4600 21750 4600
-Text GLabel 21750 4800 2    50   Output ~ 0
+Text GLabel 22800 4800 2    50   Output ~ 0
 TCK
 Text GLabel 22000 4900 2    50   Output ~ 0
@@
 P 13700 4450
 F 0 "C12" H 13815 4496 50  0000 L CNN
-F 1 "100n" H 13815 4405 50  0000 L CNN
+F 1 "10p" H 13815 4405 50  0000 L CNN
 F 2 "Capacitor_THT:C_Disc_D4.7mm_W2.5mm_P5.00mm" H 13738 4300 50  0001 C CNN
 F 3 "~" H 13700 4450 50  0001 C CNN
@@
 P 14350 4450
 F 0 "C13" H 14465 4496 50  0000 L CNN
-F 1 "100n" H 14465 4405 50  0000 L CNN
+F 1 "10p" H 14465 4405 50  0000 L CNN
 F 2 "Capacitor_THT:C_Disc_D4.7mm_W2.5mm_P5.00mm" H 14388 4300 50  0001 C CNN
 F 3 "~" H 14350 4450 50  0001 C CNN
@@
 \RST
 $Comp
-L Timer:NE555P U10
-U 1 1 5F609F15
-P 15600 10750
-F 0 "U10" H 15250 11250 50  0000 C CNN
-F 1 "NE555P" H 15350 11150 50  0000 C CNN
-F 2 "Package_DIP:DIP-8_W7.62mm" H 16250 10350 50  0001 C CNN
-F 3 "http://www.ti.com/lit/ds/symlink/ne555.pdf" H 16450 10350 50  0001 C CNN
-	1    15600 10750
-	1    0    0    -1
-$EndComp
-$Comp
 L power:GND #PWR037
 U 1 1 5F613410
@@
 Wire Wire Line
 	16100 10950 16500 10950
-Wire Wire Line
-	14500 10550 15100 10550
 Connection ~ 14500 10550
-Wire Wire Line
-	15100 10750 14500 10750
 Wire Wire Line
 	14500 10750 14500 11100
@@
 Wire Wire Line
 	14500 9700 14500 10550
-Wire Wire Line
-	15100 10950 14950 10950
-$Comp
-L power:GND #PWR035
-U 1 1 5F88C218
-P 14950 11550
-F 0 "#PWR035" H 14950 11300 50  0001 C CNN
-F 1 "GND" H 14955 11377 50  0000 C CNN
-F 2 "" H 14950 11550 50  0001 C CNN
-F 3 "" H 14950 11550 50  0001 C CNN
-	1    14950 11550
-	1    0    0    -1
-$EndComp
-Wire Wire Line
-	14950 10950 14950 11100
 $Comp
 L Device:R R24
@@
 $EndComp
 Wire Wire Line
-	14950 11400 14950 11550
-$Comp
-L Device:C C17
-U 1 1 5F94FCE8
-P 14950 11250
-F 0 "C17" H 15065 11296 50  0000 L CNN
-F 1 "10n" H 15065 11205 50  0000 L CNN
-F 2 "Capacitor_THT:C_Rect_L9.0mm_W2.5mm_P7.50mm_MKT" H 14988 11100 50  0001 C CNN
-F 3 "~" H 14950 11250 50  0001 C CNN
-F 4 "" V 14750 11300 50  0001 C CNN "Ordering Code"
-	1    14950 11250
-	1    0    0    -1
-$EndComp
-$Comp
-L MCU_Microchip_ATmega:ATmega32-16PU U7
-U 1 1 5F6BCD35
-P 12550 5150
-F 0 "U7" H 13000 7150 50  0000 C CNN
-F 1 "ATmega32-16PU" H 12100 3150 50  0000 C CNN
-F 2 "Package_DIP:DIP-40_W15.24mm" H 12550 5150 50  0001 C CIN
-F 3 "http://ww1.microchip.com/downloads/en/DeviceDoc/doc2503.pdf" H 12550 5150 50  0001 C CNN
-	1    12550 5150
-	-1   0    0    -1
-$EndComp
-Wire Wire Line
 	11500 6850 11950 6850
 Wire Wire Line
@@
 Wire Wire Line
 	14950 9950 14950 10950
-Connection ~ 14950 10950
-$Comp
-L power:GND #PWR?
+$Comp
+L power:GND #PWR01
 U 1 1 5FE8332C
 P 13000 11550
-F 0 "#PWR?" H 13000 11300 50  0001 C CNN
+F 0 "#PWR01" H 13000 11300 50  0001 C CNN
 F 1 "GND" H 13005 11377 50  0000 C CNN
 F 2 "" H 13000 11550 50  0001 C CNN
@@
 	13350 11100 13300 11100
 $Comp
-L Transistor_BJT:2N3904 Q?
+L Transistor_BJT:2N3904 Q1
 U 1 1 5FF728D8
 P 12300 11100
-F 0 "Q?" H 12250 11300 50  0000 L CNN
+F 0 "Q1" H 12250 11300 50  0000 L CNN
 F 1 "2N3904" H 12050 10950 50  0000 L CNN
-F 2 "Package_TO_SOT_THT:TO-92_Inline" H 12500 11025 50  0001 L CIN
+F 2 "Package_TO_SOT_THT:TO-92_HandSolder" H 12500 11025 50  0001 L CIN
 F 3 "https://www.fairchildsemi.com/datasheets/2N/2N3904.pdf" H 12300 11100 50  0001 L CNN
 	1    12300 11100
@@
 $EndComp
 $Comp
-L Transistor_BJT:BC328 Q?
+L Transistor_BJT:BC328 Q2
 U 1 1 5FF9EB7A
 P 13100 11100
-F 0 "Q?" H 13291 11146 50  0000 L CNN
+F 0 "Q2" H 13291 11146 50  0000 L CNN
 F 1 "BC328" H 13291 11055 50  0000 L CNN
-F 2 "Package_TO_SOT_THT:TO-92_Inline" H 13300 11025 50  0001 L CIN
+F 2 "Package_TO_SOT_THT:TO-92_HandSolder" H 13300 11025 50  0001 L CIN
 F 3 "http://www.redrok.com/PNP_BC327_-45V_-800mA_0.625W_Hfe100_TO-92.pdf" H 13100 11100 50  0001 L CNN
 	1    13100 11100
 	-1   0    0    -1
 $EndComp
+$Comp
+L MCU_Microchip_ATmega:ATmega644-20PU U7
+U 1 1 5FAB9B61
+P 12550 5150
+F 0 "U7" H 12550 3061 50  0000 C CNN
+F 1 "ATmega644-20PU" H 12550 2970 50  0000 C CNN
+F 2 "Package_DIP:DIP-40_W15.24mm" H 12550 5150 50  0001 C CIN
+F 3 "http://ww1.microchip.com/downloads/en/DeviceDoc/doc2593.pdf" H 12550 5150 50  0001 C CNN
+	1    12550 5150
+	-1   0    0    -1
+$EndComp
+$Comp
+L Device:C C19
+U 1 1 5FB12E26
+P 22500 5000
+F 0 "C19" H 22615 5046 50  0000 L CNN
+F 1 "10p" H 22615 4955 50  0000 L CNN
+F 2 "Capacitor_THT:C_Disc_D4.7mm_W2.5mm_P5.00mm" H 22538 4850 50  0001 C CNN
+F 3 "~" H 22500 5000 50  0001 C CNN
+	1    22500 5000
+	1    0    0    -1
+$EndComp
+$Comp
+L power:GND #PWR?
+U 1 1 5FB64444
+P 22500 5600
+AR Path="/5F670D5B/5FB64444" Ref="#PWR?"  Part="1"
+AR Path="/5F671D57/5FB64444" Ref="#PWR?"  Part="1"
+AR Path="/5FB64444" Ref="#PWR02"  Part="1"
+F 0 "#PWR02" H 22500 5350 50  0001 C CNN
+F 1 "GND" H 22505 5427 50  0000 C CNN
+F 2 "" H 22500 5600 50  0001 C CNN
+F 3 "" H 22500 5600 50  0001 C CNN
+	1    22500 5600
+	1    0    0    -1
+$EndComp
+Wire Wire Line
+	22500 4800 22500 4850
+Wire Wire Line
+	22500 5150 22500 5600
+Connection ~ 22500 4800
+Wire Wire Line
+	22500 4800 22800 4800
+Wire Wire Line
+	15100 10950 14950 10950
+Wire Wire Line
+	15100 10750 14500 10750
+Wire Wire Line
+	14500 10550 15100 10550
+$Comp
+L Timer:NE555P U10
+U 1 1 5F609F15
+P 15600 10750
+F 0 "U10" H 15250 11250 50  0000 C CNN
+F 1 "NE555P" H 15350 11150 50  0000 C CNN
+F 2 "Package_DIP:DIP-8_W7.62mm" H 16250 10350 50  0001 C CNN
+F 3 "http://www.ti.com/lit/ds/symlink/ne555.pdf" H 16450 10350 50  0001 C CNN
+	1    15600 10750
+	1    0    0    -1
+$EndComp
 $EndSCHEMATC

Commit message: changed MCU back to atmega32
Parts:
- removed U7: ATmega644-20PU, Package_DIP:DIP-40_W15.24mm, symbol MCU_Microchip_ATmega:ATmega644-20PU
- added U?: ATmega32-16PU, Package_DIP:DIP-40_W15.24mm, symbol MCU_Microchip_ATmega:ATmega32-16PU
Connections:
- net +5V: now also U?.10 (VCC)
- net A: now also U?.1 (PB0)
- net AREF: now also U?.32 (AREF)
- net AVCC: now also U?.30 (AVCC)
- net B: now also U?.2 (PB1)
- net C: now also U?.3 (PB2)
- net D: now also U?.4 (PB3)
- net DACH_ADC: now also U?.40 (PA0)
- net DE: now also U?.35 (PA5)
- net DH: now also U?.33 (PA7)
- net DP: now also U?.8 (PB7)
- net DZ: now also U?.34 (PA6)
- net E: now also U?.5 (PB4)
- net ENC_A: now also U?.16 (PD2)
- net ENC_B: now also U?.18 (PD4)
- net F: now also U?.6 (PB5)
- net G: now also U?.7 (PB6)
- net GND: now also U?.11 (GND), U?.31 (GND)
- net Heart_LED: now also U?.19 (PD5)
- net KE: now also U?.38 (PA2)
- net KELLER_ADC: now also U?.39 (PA1)
- net KH: now also U?.36 (PA4)
- net KZ: now also U?.37 (PA3)
- net PWM: now also U?.21 (PD7)
- net RxD: now also U?.14 (PD0)
- net SW1: now also U?.17 (PD3)
- net TCK: now also U?.24 (PC2)
- net TDI: now also U?.27 (PC5)
- net TDO: now also U?.26 (PC4)
- net TMS: now also U?.25 (PC3)
- net TxD: now also U?.15 (PD1)
- net WDI: now also U?.28 (PC6)
- net XTAL1: now also U?.13 (XTAL1)
- net XTAL2: now also U?.12 (XTAL2)
- net \RST: now also U?.9 (~RESET)
Changed lines of the file:
@@
-$EndComp
-$Comp
-L MCU_Microchip_ATmega:ATmega644-20PU U7
-U 1 1 5FAB9B61
-P 12550 5150
-F 0 "U7" H 12550 3061 50  0000 C CNN
-F 1 "ATmega644-20PU" H 12550 2970 50  0000 C CNN
-F 2 "Package_DIP:DIP-40_W15.24mm" H 12550 5150 50  0001 C CIN
-F 3 "http://ww1.microchip.com/downloads/en/DeviceDoc/doc2593.pdf" H 12550 5150 50  0001 C CNN
-	1    12550 5150
-	-1   0    0    -1
 $EndComp
 $Comp
@@
 	1    0    0    -1
 $EndComp
+$Comp
+L MCU_Microchip_ATmega:ATmega32-16PU U?
+U 1 1 5FC9465F
+P 12550 5150
+F 0 "U?" H 12550 3061 50  0000 C CNN
+F 1 "ATmega32-16PU" H 12550 2970 50  0000 C CNN
+F 2 "Package_DIP:DIP-40_W15.24mm" H 12550 5150 50  0001 C CIN
+F 3 "http://ww1.microchip.com/downloads/en/DeviceDoc/doc2503.pdf" H 12550 5150 50  0001 C CNN
+	1    12550 5150
+	-1   0    0    -1
+$EndComp
 $EndSCHEMATC
