File: Solaranlage.kicad_sch (KiCad schematic)
At the start: 117 parts, among them J1 Screw_Terminal_01x02, J2 Screw_Terminal_01x02, J3 AVR-JTAG-10, J4 USB_B, J5 USB_B, J6 Screw_Terminal_01x02, J7 Screw_Terminal_01x02, Q1 2N3904, Q2 2N3904, SW1 Rotary_Encoder_Switch_Panason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

Commit message: Rev.B -> Rev.C
Parts:
- added D15: LED_yellow_3mm, LED_THT:LED_D3.0mm, symbol Device:LED
- added R36: 330, Resistor_THT:R_Axial_DIN0204_L3.6mm_D1.6mm_P7.62mm_Horizontal, symbol Device:R
Connections:
- net GND: now also R36.2
- net pwm_ind: now reaches U12.7 (QH)
- net pwm_ind: now also D15.2 (A)
- new net: D15.1 (K), R36.1
Other:
- moved on the sheet: BZ1, Q2, R35
