File: frontplate.kicad_pcb (KiCad board)
At the start: 2 copper layers, 200 x 105 mm, 5 parts

Commit message: Rev.B -> Rev.C
Other:
- outline, holes or cut-outs redrawn
- net class Default removed
- board text added: "PWM"
